File: kicad/ble-han-port-if.kicad_sch (KiCad schematic)
At the start: 25 parts, among them J1 Conn_01x03, J2 Conn_01x04, J3 Conn_01x06, Q1 BC847, U1 ESP32-C3-WROOM-02-N4, U4 R-78B3.3-1.0 (Recom)

Commit message: Rerouted USB and fixed pos for holes
Parts:
- added R10: 0R, Resistor_SMD:R_0805_2012Metric_Pad1.20x1.40mm_HandSolder, symbol Device:R_Small
Connections:
- net TX: now also R10.2
- net D+: now reaches R4.1, U1.13 (IO18)
- net at Q1.3 (C), R7.1: now also R10.1
- net D-: now reaches R5.1, U1.14 (IO19)
Other:
- note added: "Only if Q1 mounted"
- note added: "R10 mounted only if Q1 is not needed"
Changed lines of the file:
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@@
     (title "vscp-ble-han-port-interface")
     (date "2022-10-18")
-    (rev "A")
+    (rev "B")
     (company "Grodans Paradis AB")
   )
@@
   )
   (junction (at 54.61 154.94) (diameter 0) (color 0 0 0 0)
+  )
+  (junction (at 63.5 157.48) (diameter 0) (color 0 0 0 0)
   )
   (junction (at 160.02 41.91) (diameter 0) (color 0 0 0 0)
@@
     (stroke (width 0) (type default) (color 0 0 0 0))
   )
-  (wire (pts (xy 63.5 154.94) (xy 63.5 165.1))
+  (wire (pts (xy 63.5 154.94) (xy 63.5 157.48))
     (stroke (width 0) (type default) (color 0 0 0 0))
   )
@@
     (stroke (width 0) (type default) (color 0 0 0 0))
   )
+  (wire (pts (xy 63.5 157.48) (xy 67.31 157.48))
+    (stroke (width 0) (type default) (color 0 0 0 0))
+  )
   (wire (pts (xy 44.45 167.64) (xy 54.61 167.64))
     (stroke (width 0) (type default) (color 0 0 0 0))
@@
     (stroke (width 0) (type default) (color 0 0 0 0))
   )
+  (wire (pts (xy 72.39 157.48) (xy 74.93 157.48))
+    (stroke (width 0) (type default) (color 0 0 0 0))
+  )
   (wire (pts (xy 54.61 134.62) (xy 54.61 154.94))
     (stroke (width 0) (type default) (color 0 0 0 0))
@@
     (stroke (width 0) (type default) (color 0 0 0 0))
   )
+  (wire (pts (xy 63.5 157.48) (xy 63.5 165.1))
+    (stroke (width 0) (type default) (color 0 0 0 0))
+  )
   (wire (pts (xy 74.93 176.53) (xy 74.93 170.18))
     (stroke (width 0) (type default) (color 0 0 0 0))
@@
   (polyline (pts (xy 181.61 151.13) (xy 119.38 151.13))
     (stroke (width 0) (type default) (color 0 0 0 0))
+  )
+  (text "Only if Q1\nmounted" (at 81.28 153.67 0)
+    (effects (font (size 1.27 1.27)) (justify left bottom))
+  )
+  (text "R10 mounted only if Q1 \nis not needed" (at 71.8353 155.5483 90)
+    (effects (font (size 1.27 1.27)) (justify left bottom))
   )
   (text "Debug \nInterface\n(JTAG + Serial)" (at 204.47 62.23 0)
@@
     (effects (font (size 1.27 1.27)) (justify left bottom))
   )
+  (label "D+" (at 137.16 59.69 0)
+    (effects (font (size 1.27 1.27)) (justify left bottom))
+  )
   (label "USB D+" (at 176.53 62.23 0)
     (effects (font (size 1.27 1.27)) (justify left bottom))
@@
   )
   (label "USB D-" (at 176.53 59.69 0)
+    (effects (font (size 1.27 1.27)) (justify left bottom))
+  )
+  (label "D-" (at 137.16 62.23 0)
     (effects (font (size 1.27 1.27)) (justify left bottom))
   )
@@
   (symbol (lib_id "Device:R_Small") (at 74.93 152.4 180) (unit 1)
     (in_bom yes) (on_board yes)
-    (property "Reference" "R7" (id 0) (at 73.4314 153.5684 0)
-      (effects (font (size 1.27 1.27)) (justify left))
-    )
-    (property "Value" "10k" (id 1) (at 73.4314 151.257 0)
+    (property "Reference" "R7" (id 0) (at 79.1864 153.08 0)
+      (effects (font (size 1.27 1.27)) (justify left))
+    )
+    (property "Value" "10k" (id 1) (at 80.01 151.13 0)
       (effects (font (size 1.27 1.27)) (justify left))
     )
@@
     (pin "2")
   )
+  (symbol (lib_id "Device:R_Small") (at 69.85 157.48 270) (unit 1)
+    (in_bom yes) (on_board yes)
+    (property "Reference" "R10" (id 0) (at 71.0184 158.9786 0)
+      (effects (font (size 1.27 1.27)) (justify left))
+    )
+    (property "Value" "0R" (id 1) (at 68.707 158.9786 0)
+      (effects (font (size 1.27 1.27)) (justify left))
+    )
+    (property "Footprint" "Resistor_SMD:R_0805_2012Metric_Pad1.20x1.40mm_HandSolder" (id 2) (at 69.85 157.48 0)
+      (effects (font (size 1.27 1.27)) hide)
+    )
+    (property "Datasheet" "~" (id 3) (at 69.85 157.48 0)
+      (effects (font (size 1.27 1.27)) hide)
+    )
+    (pin "1")
+    (pin "2")
+  )
   (symbol (lib_id "Regulator_Switching:R-78B3.3-2.0") (at 146.05 124.46 0) (unit 1)
     (in_bom yes) (on_board yes)
@@
       (reference "R9") (unit 1) (value "470") (footprint "Resistor_SMD:R_0805_2012Metric")
     )
+    (path "/ea834574-8109-4e39-a6eb-3c23b4eac994"
+      (reference "R10") (unit 1) (value "0R") (footprint "Resistor_SMD:R_0805_2012Metric_Pad1.20x1.40mm_HandSolder")
+    )
     (path "/652264ff-d375-48f1-9d5d-cb557ec3e3f4"
