File: kicad/ble-han-port-if.kicad_sch (KiCad schematic)
At the start: 26 parts, among them J1 Conn_01x03, J2 Conn_01x04, J3 Conn_01x06, Q1 BC847, U1 ESP32-C3-WROOM-02-N4, U4 R-78B3.3-1.0 (Recom)

Commit message: Added obis parser
Parts:
- U1: DESCRIPTION WiFi Modules (802.11) (Engineering Samples) SMD module, ESP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 -> (none)

Commit message: Added testoutput from sagemcom T211 meter
Other:
- note added: "Reservoar Capacitor 100 µF to 220 µF (mount if needed)"
- note removed: "Reservoar Capacitor (mount if needed)"
Changed lines of the file:
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@@
 		)
 	)
-	(text "Reservoar Capacitor\n(mount if needed)"
+	(text "Reservoar Capacitor\n100 µF to 220 µF\n(mount if needed)"
 		(exclude_from_sim no)
 		(at 257.81 95.25 0)
